File: nakladka_nucleo/predkosciomierz.brd (EAGLE design)
At the start: 80 x 70 mm, 22 parts, among them IC3 LD117AS28TR, SW1 SCHURTER-LSH-1301.9320, SW2 SCHURTER-LSH-1301.9320, SW3 SCHURTER-LSH-1301.9320, SW4 SCHURTER-LSH-1301.9320, SW5 C&K_OS102011MA1QN1C&K_OS10201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, SW6 C&K_OS102011MA1QN1C&K_OS10201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, X1 NEB21R

Commit message: Add files via upload
Parts:
- removed D1: 1N4004, diode:DO41-10
- removed IC3: LD117AS28TR, v-reg:SOT223
- removed JP6: (no value), pinhead:1X09
- added C5, C6, C7, C8, C9: 100n, rcl:C1206
- added JP10: (no value), pinhead:1X06
- added JP3: (no value), moduly:1X09
- added JP9: (no value), pinhead:1X02
- added LED2: (no value), led:LED5MM
- added R2: 1k, rcl:0207/2V
- added R3, R4, R5: 1M, rcl:0207/2V
- C1, C4: device rcl:C1210 -> rcl:C1206
- C2, C3: value 10u -> 47u; device rcl:E2-5 -> rcl:PANASONIC_D
- JP5: device pinhead:1X06 -> moduly:1X05
- R1: device rcl:0204/7 -> rcl:0207/2V
- SW1, SW2, SW3, SW4: value SCHURTER-LSH-1301.9320 -> (none)
- moved C1 51.9 mm to (26.0, 66.0), turned to 270 degrees
- moved C3 26.8 mm to (31.4, 12.2), flipped to the bottom, turned to 270 degrees
- moved C4 25.5 mm to (14.8, 30.3), turned to 180 degrees
- moved C2 21.3 mm to (15.9, 35.2), flipped to the bottom, turned to 0 degrees
- moved JP4 21.2 mm to (13.4, 41.2), flipped to the bottom, turned to 0 degrees
- moved JP5 12.7 mm to (40.2, 31.5)
- moved LED1 6.37 mm to (11.7, 5.20)
- moved R1 4.05 mm to (10.9, 9.66), turned to 0 degrees
- moved X1 1.27 mm to (6.10, 60.0)
- moved SW3 1.09 mm to (24.9, 46.3)
- moved SW5 1.02 mm to (22.0, 7.17)
- moved SW4 0.57 mm to (33.0, 54.0)
- moved SW1 0.41 mm to (24.9, 62.1)
- moved SW2 0.40 mm to (16.8, 54.0)
- moved JP7 0.30 mm to (52.1, 30.6)
Connections:
- removed net N$3: D1.C, SW5.3
- removed net PA5_B4: JP2.11, SW4.NO2
- removed net PB8_B2: JP2.3, SW2.NO1
- removed net PB9_B3: JP2.5, SW3.NO1
- removed net PC12: JP1.3
- removed net PC5: JP2.6
- removed net PC9_B1: JP2.1, SW1.NO1
- new net EN: JP4.2
- new net EN_B: JP10.6
- new net N$5: R4.2, R5.1
- new net PA5_B4_BACK: JP2.11, SW4.NO1, SW4.NO2
- new net PB8_B2_ENTER: JP2.3, SW2.NO1, SW2.NO2
- new net PB9_B3_PREV: JP2.5, SW3.NO1, SW3.NO2
- new net PC12_D_BAT: JP1.3, LED2.A
- new net PC5_ADC: C1.1, JP2.6, JP9.1, R3.2, R4.1
- new net PC9_B1_NEXT: JP2.1, SW1.NO1, SW1.NO2
- new net PG: JP4.1
- new net PPS: JP5.1
- new net STATE: JP10.1
- new net VIN_NUCLEO: JP1.24
- net +3.3V: now also C5.1, C6.1, C7.1, JP3.1, JP5.5; no longer JP4.5, JP6.1
- net +5V_IN: now also C8.1, JP10.5; no longer JP5.5
- net E5V: now also C9.1, JP4.5; no longer C4.1, IC3.4
- net GND: now also C5.2, C6.2, C7.2, C8.2, C9.2, JP10.4, JP3.2, JP9.2, R2.1, R3.1, SW1.C1, SW2.C1, SW3.C1, SW4.C1; no longer IC3.1, JP1.19, JP2.20, JP2.9, JP6.2
- net N$2: now also SW5.3, X1.1; no longer C1.1, C2.+, IC3.3, SW5.2
- net N$4: now also LED2.K, R2.2; no longer D1.A, X1.1
- net PA0_B_RXD: now also JP10.2; no longer JP5.2
- net PA1_B_TXD: now also JP10.3; no longer JP5.3
- net PA6_SDIO_CD: now also JP3.9; no longer JP6.9
- net PB2_SDIO_CLK: now also JP3.5; no longer JP6.5
- net PC10_GPS_RX: now also JP5.2; no longer JP4.2
- net PC11_GPS_TX: now also JP5.3; no longer JP4.3
- net PC8_SDIO_D0: now also JP3.3; no longer JP6.3
- net PD2_SDIO_CMD: now also JP3.4; no longer JP6.4
- net VIN: now also C2.+, C4.1, JP4.3, R5.2, SW5.2; no longer JP1.24
Routing:
- net VIN: track 0.00 -> 66.5 mm
- net PC5_ADC: track 0.00 -> 48.4 mm
- net N$4: track 50.7 -> 3.74 mm
- net +3.3V: track 105.4 -> 69.2 mm
- net PB8_B2_ENTER: track 0.00 -> 34.7 mm
- net N$2: track 36.2 -> 68.4 mm
- net PC12_D_BAT: track 0.00 -> 30.7 mm
- net PB9_B3_PREV: track 0.00 -> 30.4 mm
- net GND: track 26.9 -> 0.00 mm
- net PA5_B4_BACK: track 0.00 -> 22.6 mm
- net PB9_B3: track 21.7 -> 0.00 mm
- net PA5_B4: track 20.5 -> 0.00 mm
- net N$3: track 19.9 -> 0.00 mm
- net PB8_B2: track 19.1 -> 0.00 mm
- net PA1_B_TXD: track 46.6 -> 28.6 mm
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Other:
- board text added: "IN"
- board text added: "Luiza Blaszczak Praca inzynierska Predkosciomierz"
- board text added: "OUT"
- board text added: "PG"
- board text removed: "Luiza Błaszczak Praca inżynierska Prędkościomierz"
