File: nakladka_nucleo/predkosciomierz.sch (EAGLE design)
At the start: 22 parts, among them IC3 LD117AS28TR, SW1 SCHURTER-LSH-1301.9320, SW2 SCHURTER-LSH-1301.9320, SW3 SCHURTER-LSH-1301.9320, SW4 SCHURTER-LSH-1301.9320, SW5 C&K_OS102011MA1QN1C&K_OS10201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, SW6 C&K_OS102011MA1QN1C&K_OS10201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, X1 NEB21R

Commit message: Add files via upload
Parts:
- removed D1: 1N4004, diode:1N4004
- removed IC3: LD117AS28TR, v-reg:LD117AS28TR
- removed JP6: (no value), pinhead:PINHD-1X9
- added C5, C6, C7, C8, C9: 100n, rcl:C-EUC1206
- added JP10: (no value), pinhead:PINHD-1X6
- added JP3: (no value), moduly:PINHD-1X9
- added JP9: (no value), pinhead:PINHD-1X2
- added LED2: (no value), led:LED5MM
- added R2: 1k, rcl:R-EU_0207/2V
- added R3, R4, R5: 1M, rcl:R-EU_0207/2V
- C1, C4: device rcl:C-EUC1210 -> rcl:C-EUC1206
- C2, C3: value 10u -> 47u; device rcl:CPOL-EUE2-5 -> rcl:CPOL-EUD
- JP5: device pinhead:PINHD-1X6 -> moduly:PINHD-1X5
- R1: device rcl:R-EU_0204/7 -> rcl:R-EU_0207/2V
Connections:
- removed net N$3: D1.C, SW5.3
- removed net PA5_B4: JP2.11, SW4.NO@2
- removed net PB8_B2: JP2.3, SW2.NO@1
- removed net PB9_B3: JP2.5, SW3.NO@1
- removed net PC12: JP1.3
- removed net PC5: JP2.6
- removed net PC9_B1: JP2.1, SW1.NO@1
- new net EN: JP4.2
- new net EN_B: JP10.6
- new net N$5: R4.2, R5.1
- new net PA5_B4_BACK: JP2.11, SW4.NO@1, SW4.NO@2
- new net PB8_B2_ENTER: JP2.3, SW2.NO@1, SW2.NO@2
- new net PB9_B3_PREV: JP2.5, SW3.NO@1, SW3.NO@2
- new net PC12_D_BAT: JP1.3, LED2.A
- new net PC5_ADC: C1.1, JP2.6, JP9.1, R3.2, R4.1
- new net PC9_B1_NEXT: JP2.1, SW1.NO@1, SW1.NO@2
- new net PG: JP4.1
- new net PPS: JP5.1
- new net STATE: JP10.1
- new net VIN_NUCLEO: JP1.24
- net +3.3V: now also C5.1, C6.1, C7.1, JP3.1, JP5.5; no longer JP4.5, JP6.1
- net +5V_IN: now also C8.1, JP10.5; no longer JP5.5
- net E5V: now also C9.1, JP4.5; no longer C4.1, IC3.OUT
- net GND: now also C5.2, C6.2, C7.2, C8.2, C9.2, JP10.4, JP3.2, JP9.2, R2.1, R3.1, SW1.C@1, SW2.C@1, SW3.C@1, SW4.C@1; no longer IC3.ADJ, JP1.19, JP2.20, JP2.9, JP6.2
- net N$2: now also SW5.3, X1.1; no longer C1.1, C2.+, IC3.IN, SW5.2
- net N$4: now also LED2.C, R2.2; no longer D1.A, X1.1
- net PA0_B_RXD: now also JP10.2; no longer JP5.2
- net PA1_B_TXD: now also JP10.3; no longer JP5.3
- net PA6_SDIO_CD: now also JP3.9; no longer JP6.9
- net PB2_SDIO_CLK: now also JP3.5; no longer JP6.5
- net PC10_GPS_RX: now also JP5.2; no longer JP4.2
- net PC11_GPS_TX: now also JP5.3; no longer JP4.3
- net PC8_SDIO_D0: now also JP3.3; no longer JP6.3
- net PD2_SDIO_CMD: now also JP3.4; no longer JP6.4
- net VIN: now also C2.+, C4.1, JP4.3, R5.2, SW5.2; no longer JP1.24
Other:
- note added: "FILTRACJA ZASILANIA"
- note added: "S9V11F3S5CMA"
- moved on the sheet: C2, C3, C4, LED1, R1, SW5, X1
